File: hardware/conductivity.kicad_sch (KiCad schematic)
At the start: 7 parts, among them J2 PAD1, J3 PAD2, Q1 2N3904

Commit message: prod stuff
Parts:
- BT5: LCSC (none) -> C70376
- D1: LCSC (none) -> C52034661
- Q1: LCSC (none) -> C2874602
- R6: footprint Resistor_THT:R_Axial_DIN0207_L6.3mm_D2.5mm_P7.62mm_Horizontal -> Resistor_THT:R_Axial_DIN0204_L3.6mm_D1.6mm_P5.08mm_Horizontal; LCSC (none) -> C2848520
- R7: footprint Resistor_THT:R_Axial_DIN0207_L6.3mm_D2.5mm_P7.62mm_Horizontal -> Resistor_THT:R_Axial_DIN0204_L3.6mm_D1.6mm_P5.08mm_Horizontal; LCSC (none) -> C2896925
Changed lines of the file:
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@@
+			)
+		)
+		(property "LCSC" "C70376"
+			(at 162.56 90.17 0)
+			(hide yes)
+			(show_name no)
+			(do_not_autoplace no)
+			(effects
+				(font
+					(size 1.27 1.27)
+				)
 			)
 		)
@@
 			)
 		)
-		(property "Footprint" "Resistor_THT:R_Axial_DIN0207_L6.3mm_D2.5mm_P7.62mm_Horizontal"
+		(property "Footprint" "Resistor_THT:R_Axial_DIN0204_L3.6mm_D1.6mm_P5.08mm_Horizontal"
 			(at 139.7 91.44 0)
 			(hide yes)
@@
 		)
 		(property "Description" "Resistor, small US symbol"
+			(at 139.7 91.44 0)
+			(hide yes)
+			(show_name no)
+			(do_not_autoplace no)
+			(effects
+				(font
+					(size 1.27 1.27)
+				)
+			)
+		)
+		(property "LCSC" "C2848520"
 			(at 139.7 91.44 0)
 			(hide yes)
@@
 		)
 		(property "Sim.Pins" "1=E 2=B 3=C"
+			(at 144.78 88.9 0)
+			(hide yes)
+			(show_name no)
+			(do_not_autoplace no)
+			(effects
+				(font
+					(size 1.27 1.27)
+				)
+			)
+		)
+		(property "LCSC" "C2874602"
 			(at 144.78 88.9 0)
 			(hide yes)
@@
 			)
 		)
-		(property "Footprint" "Resistor_THT:R_Axial_DIN0207_L6.3mm_D2.5mm_P7.62mm_Horizontal"
+		(property "Footprint" "Resistor_THT:R_Axial_DIN0204_L3.6mm_D1.6mm_P5.08mm_Horizontal"
 			(at 130.81 88.9 0)
 			(hide yes)
@@
 		(property "Description" "Resistor, small US symbol"
 			(at 130.81 88.9 0)
+			(hide yes)
+			(show_name no)
+			(do_not_autoplace no)
+			(effects
+				(font
+					(size 1.27 1.27)
+				)
+			)
+		)
+		(property "LCSC" "C2896925"
+			(at 130.81 88.9 90)
 			(hide yes)
 			(show_name no)
@@
 			(at 154.94 82.55 0)
 			(hide yes)
+			(show_name no)
+			(do_not_autoplace no)
+			(effects
+				(font
+					(size 1.27 1.27)
+				)
+			)
+		)
+		(property "LCSC" "C52034661"
+			(at 154.94 82.55 0)
+			(hide yes)
