File: hardware/continuity.kicad_sch (KiCad schematic)
At the start: 3 parts, among them J1 PROBE

Commit message: prod stuff
Parts:
- BT3: LCSC (none) -> C70376
- BZ1: LCSC (none) -> C49246930
Changed lines of the file:
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@@
+			)
+		)
+		(property "LCSC" "C70376"
+			(at 128.27 81.28 0)
+			(hide yes)
+			(show_name no)
+			(do_not_autoplace no)
+			(effects
+				(font
+					(size 1.27 1.27)
+				)
 			)
 		)
@@
 			(at 153.67 80.01 0)
 			(hide yes)
+			(show_name no)
+			(do_not_autoplace no)
+			(effects
+				(font
+					(size 1.27 1.27)
+				)
+			)
+		)
+		(property "LCSC" "C49246930"
+			(at 153.67 80.01 0)
+			(hide yes)
